File: elec/layout/default/octoknob.kicad_pcb (KiCad board)
At the start: 2 copper layers, 143.6 x 35.3 mm, 52 parts

Commit message: saves changes
Other:
- board outline removed
Changed lines of the file:
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@@
       (net 3 "ring.led_1-vdd") (pintype "stereo") (solder_mask_margin 0.1016) (thermal_bridge_angle 45))
   )
-  (gr_line (start 82.042 89.154) (end 225.679 89.154)
-    (stroke (width 0.1) (type default)) (layer "Edge.Cuts"))
-  (gr_line (start 82.042 89.154) (end 82.042 124.46)
-    (stroke (width 0.1) (type default)) (layer "Edge.Cuts"))
-  (gr_line (start 82.042 124.46) (end 225.679 124.46)
-    (stroke (width 0.1) (type default)) (layer "Edge.Cuts"))
-  (gr_line (start 225.679 89.154) (end 225.679 124.46)
-    (stroke (width 0.1) (type default)) (layer "Edge.Cuts"))
   (group "" (id 08ffc31c-5b61-42c3-84ba-78607af77dfb)
     (members
